File: hardware/cantor-pro-lp-pcb.kicad_pcb (KiCad board)
At the start: 2 copper layers, 133.4 x 89.9 mm, 42 parts, among them J1 TRRS, J2 BAT, K00 KEYSW, K01 KEYSW, K02 KEYSW, K03 KEYSW, K04 KEYSW, K05 KEYSW, K10 KEYSW, K11 KEYSW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

Commit message: Custom Message
Other:
- board text added: "MADE BY ME"
- board text removed: "MADE BY MANUEL"
